File: KiCAD/Hyperdrive!.sch (KiCad schematic (older format))
At the start: 62 parts, among them CON1 USB-MINI-B, K1 SPRI/O, P1 RIR PCB, P2 ICSP, P3 Display PCB, P4 Motor Feedback PCB, P5 Extra I/Os, P7 PWR, U1 24AA256, U2 LD39200, U3 LT3464, U4 DSPIC33EP512GM706, U5 FT201X, X1 16MHz

Commit message: Updated 3D-Model, and PCBs.
Parts:
- added D4: LED, ~, symbol LED
- added P8: I2C, symbol CONN_4
- added P9: PWR, symbol CONN_2
- added R16: R, ~, symbol R
- added TP1, TP10, TP11, TP2, TP3, TP4, TP5, TP6, TP7, TP8, TP9: TP, symbol TP
Connections:
- wire segments 303 -> 319
Other:
- note added: "Extra Connectors"
- note added: "PWR LED\n"
- moved on the sheet: P7
