File: KiCAD/file551E8A3A.sch (KiCad schematic (older format))
At the start: 13 parts, among them P6 EDG_SEN, U6 GP2Y0A51SK0F, U7 LSM330, U8 GP2Y0E03

Commit message: Updated 3D-Model, and PCBs.
Parts:
- added TP12, TP13, TP14, TP15, TP16, TP17, TP18: TP, symbol TP
Connections:
- wire segments 64 -> 72
Other:
- moved on the sheet: C24, C26, C27, C28, C30, U7
